Commit message: fix(myagv_plus_description): Add ros2_control functionality

File: myagv_plus_description/urdf/common/gazebo.urdf.xacro (robot description, xacro)
@@ -1,12 +1,73 @@
 <?xml version="1.0" encoding="utf-8"?>
 <robot xmlns:xacro="http://www.ros.org/wiki/xacro">
-  <!-- base defining macro -->
-  <xacro:macro name="base" params="wheel_radius namespace">
-    <link name="${namespace}base_footprint"/>
-  <joint name="${namespace}base_joint" type="fixed">
-    <parent link="${namespace}base_footprint"/>
-    <child link="${namespace}base_link" />
-    <origin xyz="0 0 ${wheel_radius}" rpy="0 0 0"/>
-  </joint>
+  <xacro:macro name="controller" params="config_file namespace:=''">
+    <gazebo>
+      <plugin filename="ign_ros2_control-system" name="ign_ros2_control::IgnitionROS2ControlPlugin">
+        <controller_manager_name>controller_manager</controller_manager_name>
+        <parameters>${config_file}</parameters>
+        <ros>
+          <namespace>${namespace}</namespace>
+          <remapping>imu_broadcaster/imu:=imu/data</remapping>
+          <remapping>imu_broadcaster/transition_event:=_imu_broadcaster/transition_event</remapping>
+          <remapping>joint_state_broadcaster/transition_event:=_joint_state_broadcaster/transition_event</remapping>
+          <remapping>mecanum_drive_controller/cmd_vel_unstamped:=cmd_vel</remapping>
+          <remapping>mecanum_drive_controller/odom:=odometry/wheels</remapping>
+          <remapping>mecanum_drive_controller/transition_event:=_mecanum_drive_controller/transition_event</remapping>
+          <remapping>/diagnostics:=diagnostics</remapping>
+          <remapping>/tf:=tf</remapping>
+          <remapping>/tf_static:=tf_static</remapping>
+        </ros>
+      </plugin>
+    </gazebo>
+  </xacro:macro>
+  <!-- Gauss noise macro -->
+  <xacro:macro name="gauss_noise"
+    params="mean:=0.0 stddev:=0.0 bias_mean:=0.0 bias_stddev:=0.0 precision:=0.0">
+    <noise type="gaussian">
+      <mean>${mean}</mean>
+      <stddev>${stddev}</stddev>
+      <bias_mean>${bias_mean}</bias_mean>
+      <bias_stddev>${bias_stddev}</bias_stddev>
+      <precision>${precision}</precision>
+    </noise>
+  </xacro:macro>
+  <xacro:macro name="imu" params="reference_frame namespace:=''">
+    <xacro:property name="ns" value="${namespace + '/' if namespace != '' else ''}" />
+    <gazebo reference="${reference_frame}">
+      <sensor name="${ns}imu" type="imu">
+        <always_on>true</always_on>
+        <update_rate>25</update_rate>
+        <topic>${ns}imu/data_raw</topic>
+        <visualize>false</visualize>
+        <enable_metrics>false</enable_metrics>
+        <ignition_frame_id>imu_link</ignition_frame_id>
+        <imu>
+          <angular_velocity>
+            <!-- rad/s | no bias_mean in datasheet -->
+            <x>
+              <xacro:gauss_noise stddev="5.24e-3" bias_mean="2.0e-3" precision="1.07e-3" />
+            </x>
+            <y>
+              <xacro:gauss_noise stddev="5.24e-3" bias_mean="2.0e-3" precision="1.07e-3" />
+            </y>
+            <z>
+              <xacro:gauss_noise stddev="5.24e-3" bias_mean="2.0e-3" precision="1.07e-3" />
+            </z>
+          </angular_velocity>
+          <linear_acceleration>
+            <!-- m/s^2 | no bias_mean in datasheet -->
+            <x>
+              <xacro:gauss_noise stddev="1.86e-3" bias_mean="1.0e-3" precision="2.40e-3" />
+            </x>
+            <y>
+              <xacro:gauss_noise stddev="1.86e-3" bias_mean="1.0e-3" precision="2.40e-3" />
+            </y>
+            <z>
+              <xacro:gauss_noise stddev="1.86e-3" bias_mean="1.0e-3" precision="2.40e-3" />
+            </z>
+          </linear_acceleration>
+        </imu>
+      </sensor>
+    </gazebo>
   </xacro:macro>
 </robot>

File: myagv_plus_description/urdf/common/ros2_control.urdf.xacro (robot description, xacro)
@@ -1,12 +1,98 @@
 <?xml version="1.0" encoding="utf-8"?>
 <robot xmlns:xacro="http://www.ros.org/wiki/xacro">
-  <!-- base defining macro -->
-  <xacro:macro name="base" params="wheel_radius namespace">
-    <link name="${namespace}base_footprint"/>
-  <joint name="${namespace}base_joint" type="fixed">
-    <parent link="${namespace}base_footprint"/>
-    <child link="${namespace}base_link" />
-    <origin xyz="0 0 ${wheel_radius}" rpy="0 0 0"/>
-  </joint>
+  <xacro:macro name="imu" params="name:='imu' namespace:=''" >
+    <xacro:property name="ns" value="${namespace + '/' if namespace != '' else ''}" />
+    <ros2_control name="${ns}${name}" type="sensor">
+      <hardware>
+        <plugin>rosbot_hardware_interfaces/RosbotImuSensor</plugin>
+        <param name="connection_timeout_ms">30000</param>
+        <param name="connection_check_period_ms">1000</param>
+      </hardware>
+      <sensor name="${ns}imu">
+        <state_interface name="orientation.x" />
+        <state_interface name="orientation.y" />
+        <state_interface name="orientation.z" />
+        <state_interface name="orientation.w" />
+        <state_interface name="angular_velocity.x" />
+        <state_interface name="angular_velocity.y" />
+        <state_interface name="angular_velocity.z" />
+        <state_interface name="linear_acceleration.x" />
+        <state_interface name="linear_acceleration.y" />
+        <state_interface name="linear_acceleration.z" />
+      </sensor>
+    </ros2_control>
+  </xacro:macro>
+  <xacro:macro name="rosbot_system" params="name:='rosbot_system' namespace:=''" >
+    <xacro:property name="ns" value="${namespace + '/' if namespace != '' else ''}" />
+    <ros2_control name="${ns}${name}" type="system">
+      <hardware>
+        <plugin>rosbot_hardware_interfaces/RosbotSystem</plugin>
+        <param name="connection_timeout_ms">30000</param>
+        <param name="connection_check_period_ms">1000</param>
+        <param name="velocity_command_joint_order">
+          rb_wheel_joint, lb_wheel_joint, rf_wheel_joint, lf_wheel_joint
+        </param>
+      </hardware>
+      <joint name="lf_wheel_joint">
+        <command_interface name="velocity" />
+        <state_interface name="position" />
+        <state_interface name="velocity" />
+      </joint>
+      <joint name="rf_wheel_joint">
+        <command_interface name="velocity" />
+        <state_interface name="position" />
+        <state_interface name="velocity" />
+      </joint>
+      <joint name="lb_wheel_joint">
+        <command_interface name="velocity" />
+        <state_interface name="position" />
+        <state_interface name="velocity" />
+      </joint>
+      <joint name="rb_wheel_joint">
+        <command_interface name="velocity" />
+        <state_interface name="position" />
+        <state_interface name="velocity" />
+      </joint>
+    </ros2_control>
+  </xacro:macro>
+  <xacro:macro name="gz_rosbot_system" params="name:='rosbot_system' namespace:=''" >
+    <xacro:property name="ns" value="${namespace + '/' if namespace != '' else ''}" />
+    <ros2_control name="${ns}${name}" type="system">
+      <hardware>
+        <plugin>gz_ros2_control/GazeboSimSystem</plugin>
+      </hardware>
+      <joint name="lf_wheel_joint">
+        <command_interface name="velocity" />
+        <state_interface name="position" />
+        <state_interface name="velocity" />
+      </joint>
+      <joint name="rf_wheel_joint">
+        <command_interface name="velocity" />
+        <state_interface name="position" />
+        <state_interface name="velocity" />
+      </joint>
+      <joint name="lb_wheel_joint">
+        <command_interface name="velocity" />
+        <state_interface name="position" />
+        <state_interface name="velocity" />
+      </joint>
+      <joint name="rb_wheel_joint">
+        <command_interface name="velocity" />
+        <state_interface name="position" />
+        <state_interface name="velocity" />
+      </joint>
+      <sensor name="${ns}imu">
+        <state_interface name="orientation.x" />
+        <state_interface name="orientation.y" />
+        <state_interface name="orientation.z" />
+        <state_interface name="orientation.w" />
+        <state_interface name="angular_velocity.x" />
+        <state_interface name="angular_velocity.y" />
+        <state_interface name="angular_velocity.z" />
+        <state_interface name="linear_acceleration.x" />
+        <state_interface name="linear_acceleration.y" />
+        <state_interface name="linear_acceleration.z" />
+      </sensor>
+    </ros2_control>
   </xacro:macro>
 </robot>
