Commit message: fix(myagv_plus_description): Update the urdf.xacro file

File: myagv_plus_description/urdf/common/ros2_control.urdf.xacro (robot description, xacro)
@@ -1,26 +1,4 @@
 <?xml version="1.0" encoding="utf-8"?>
 <robot xmlns:xacro="http://www.ros.org/wiki/xacro">
-  <xacro:macro name="imu" params="name:='imu' namespace:=''" >
-    <xacro:property name="ns" value="${namespace + '/' if namespace != '' else ''}" />
-    <ros2_control name="${ns}${name}" type="sensor">
-      <hardware>
-        <plugin>rosbot_hardware_interfaces/RosbotImuSensor</plugin>
-        <param name="connection_timeout_ms">30000</param>
-        <param name="connection_check_period_ms">1000</param>
-      </hardware>
-      <sensor name="${ns}imu">
-        <state_interface name="orientation.x" />
-        <state_interface name="orientation.y" />
-        <state_interface name="orientation.z" />
-        <state_interface name="orientation.w" />
-        <state_interface name="angular_velocity.x" />
-        <state_interface name="angular_velocity.y" />
-        <state_interface name="angular_velocity.z" />
-        <state_interface name="linear_acceleration.x" />
-        <state_interface name="linear_acceleration.y" />
-        <state_interface name="linear_acceleration.z" />
-      </sensor>
-    </ros2_control>
-  </xacro:macro>
   <xacro:macro name="rosbot_system" params="name:='rosbot_system' namespace:=''" >
     <xacro:property name="ns" value="${namespace + '/' if namespace != '' else ''}" />
@@ -54,4 +32,16 @@
         <state_interface name="velocity" />
       </joint>
+      <sensor name="${ns}imu">
+        <state_interface name="orientation.x" />
+        <state_interface name="orientation.y" />
+        <state_interface name="orientation.z" />
+        <state_interface name="orientation.w" />
+        <state_interface name="angular_velocity.x" />
+        <state_interface name="angular_velocity.y" />
+        <state_interface name="angular_velocity.z" />
+        <state_interface name="linear_acceleration.x" />
+        <state_interface name="linear_acceleration.y" />
+        <state_interface name="linear_acceleration.z" />
+      </sensor>
     </ros2_control>
   </xacro:macro>

File: myagv_plus_description/urdf/myagv_plus.urdf.xacro (robot description, xacro)
@@ -14,11 +14,10 @@
   <xacro:base.body wheel_radius="${wheel_radius}" namespace="${namespace}" />
   <!-- WHEEL -->
-  <xacro:wheel.wheel wheel_radius="${wheel_radius}" side="lf" mecanum="${mecanum}" />
-  <xacro:wheel.wheel wheel_radius="${wheel_radius}" side="lb" mecanum="${mecanum}" />
-  <xacro:wheel.wheel wheel_radius="${wheel_radius}" side="rf" mecanum="${mecanum}" />
-  <xacro:wheel.wheel wheel_radius="${wheel_radius}" side="rb" mecanum="${mecanum}" />
+  <xacro:wheel.wheel wheel_radius="${wheel_radius}" side="fl" mecanum="${mecanum}" />
+  <xacro:wheel.wheel wheel_radius="${wheel_radius}" side="rl" mecanum="${mecanum}" />
+  <xacro:wheel.wheel wheel_radius="${wheel_radius}" side="fr" mecanum="${mecanum}" />
+  <xacro:wheel.wheel wheel_radius="${wheel_radius}" side="rr" mecanum="${mecanum}" />
   <!-- HARDWARE PLUGINS -->
   <xacro:unless value="${use_sim}">
-    <xacro:ros2_control.imu namespace="${namespace}" />
     <xacro:ros2_control.rosbot_system namespace="${namespace}" />
   </xacro:unless>

File: myagv_plus_description/urdf/robot/wheel.urdf.xacro (robot description, xacro)
@@ -10,34 +10,29 @@
     <xacro:property name="iyy" value="0.000067" />
     <xacro:property name="izz" value="0.000041" />
-    <!-- <xacro:property name="x" value="0.0" />
-    <xacro:property name="y" value="0.0" />
-    <xacro:property name="mesh" value="" />
-    <xacro:property name="visual_rotation" value="0.0" />
-    <xacro:property name="fdir" value="1.0 0.0 0.0" /> -->
-    <xacro:if value="${side == 'lf'}">
+    <xacro:if value="${side == 'fl'}">
       <xacro:property name="x" value="${wheel_separation_x/2.0}" />
       <xacro:property name="y" value="${wheel_separation_y/2.0}" />
-      <xacro:property name="mesh" value="package://myagv_plus_description/meshes/wheel_lf_link.stl" />
+      <xacro:property name="mesh" value="package://myagv_plus_description/meshes/wheel_fl_link.stl" />
       <xacro:property name="visual_rotation" value="${pi}" />
       <xacro:property name="fdir" value="1.0 -1.0 0.0" />
     </xacro:if>
-    <xacro:if value="${side == 'rf'}">
+    <xacro:if value="${side == 'fr'}">
       <xacro:property name="x" value="${wheel_separation_x/2.0}" />
       <xacro:property name="y" value="${-wheel_separation_y/2.0}" />
-      <xacro:property name="mesh" value="package://myagv_plus_description/meshes/wheel_rf_link.stl" />
+      <xacro:property name="mesh" value="package://myagv_plus_description/meshes/wheel_fr_link.stl" />
       <xacro:property name="visual_rotation" value="${pi}" />
       <xacro:property name="fdir" value="1.0 1.0 0.0" />
     </xacro:if>
-    <xacro:if value="${side == 'lb'}">
+    <xacro:if value="${side == 'rl'}">
       <xacro:property name="x" value="${-wheel_separation_x/2.0}" />
       <xacro:property name="y" value="${wheel_separation_y/2.0}" />
-      <xacro:property name="mesh" value="package://myagv_plus_description/meshes/wheel_lb_link.stl" />
+      <xacro:property name="mesh" value="package://myagv_plus_description/meshes/wheel_rl_link.stl" />
       <xacro:property name="visual_rotation" value="${0.0}" />
       <xacro:property name="fdir" value="1.0 1.0 0.0" />
     </xacro:if>
-    <xacro:if value="${side == 'rb'}">
+    <xacro:if value="${side == 'rr'}">
       <xacro:property name="x" value="${-wheel_separation_x/2.0}" />
       <xacro:property name="y" value="${-wheel_separation_y/2.0}" />
-      <xacro:property name="mesh" value="package://myagv_plus_description/meshes/wheel_rb_link.stl" />
+      <xacro:property name="mesh" value="package://myagv_plus_description/meshes/wheel_rr_link.stl" />
       <xacro:property name="visual_rotation" value="${0.0}" />
       <xacro:property name="fdir" value="1.0 -1.0 0.0" />

Commit message: feat(hardware_interfaces): add ros2_control system interface for MyAGV Plus

File: myagv_plus_description/urdf/common/ros2_control.urdf.xacro (robot description, xacro)
@@ -5,30 +5,35 @@
     <ros2_control name="${ns}${name}" type="system">
       <hardware>
-        <plugin>rosbot_hardware_interfaces/RosbotSystem</plugin>
-        <param name="connection_timeout_ms">30000</param>
-        <param name="connection_check_period_ms">1000</param>
-        <param name="velocity_command_joint_order">
-          rb_wheel_joint, lb_wheel_joint, rf_wheel_joint, lf_wheel_joint
-        </param>
+        <plugin>myagvplus_hardware_interfaces/MyAGVPlusInterface</plugin>
+        <param name="port">/dev/ttyACM0</param>
+        <param name="baudrate">921600</param>
       </hardware>
-      <joint name="lf_wheel_joint">
+      <joint name="fl_wheel_joint">
         <command_interface name="velocity" />
         <state_interface name="position" />
         <state_interface name="velocity" />
+        <param name="can_id">0x01</param>
+        <param name="mst_id">0x11</param>
       </joint>
-      <joint name="rf_wheel_joint">
+      <joint name="fr_wheel_joint">
         <command_interface name="velocity" />
         <state_interface name="position" />
         <state_interface name="velocity" />
+        <param name="can_id">0x02</param>
+        <param name="mst_id">0x12</param>
       </joint>
-      <joint name="lb_wheel_joint">
+      <joint name="rl_wheel_joint">
         <command_interface name="velocity" />
         <state_interface name="position" />
         <state_interface name="velocity" />
+        <param name="can_id">0x03</param>
+        <param name="mst_id">0x13</param>
       </joint>
-      <joint name="rb_wheel_joint">
+      <joint name="rr_wheel_joint">
         <command_interface name="velocity" />
         <state_interface name="position" />
         <state_interface name="velocity" />
+        <param name="can_id">0x04</param>
+        <param name="mst_id">0x14</param>
       </joint>
       <sensor name="${ns}imu">

Commit message: feat(ros2_control): unify ros2_control bringup for real hardware and Gazebo simulation

File: myagv_plus_description/urdf/common/ros2_control.urdf.xacro (robot description, xacro)
@@ -37,16 +37,4 @@
         <param name="mst_id">0x14</param>
       </joint>
-      <sensor name="${ns}imu">
-        <state_interface name="orientation.x" />
-        <state_interface name="orientation.y" />
-        <state_interface name="orientation.z" />
-        <state_interface name="orientation.w" />
-        <state_interface name="angular_velocity.x" />
-        <state_interface name="angular_velocity.y" />
-        <state_interface name="angular_velocity.z" />
-        <state_interface name="linear_acceleration.x" />
-        <state_interface name="linear_acceleration.y" />
-        <state_interface name="linear_acceleration.z" />
-      </sensor>
     </ros2_control>
   </xacro:macro>
@@ -57,20 +45,20 @@
         <plugin>gz_ros2_control/GazeboSimSystem</plugin>
       </hardware>
-      <joint name="lf_wheel_joint">
+      <joint name="fl_wheel_joint">
         <command_interface name="velocity" />
         <state_interface name="position" />
         <state_interface name="velocity" />
       </joint>
-      <joint name="rf_wheel_joint">
+      <joint name="fr_wheel_joint">
         <command_interface name="velocity" />
         <state_interface name="position" />
         <state_interface name="velocity" />
       </joint>
-      <joint name="lb_wheel_joint">
+      <joint name="rl_wheel_joint">
         <command_interface name="velocity" />
         <state_interface name="position" />
         <state_interface name="velocity" />
       </joint>
-      <joint name="rb_wheel_joint">
+      <joint name="rr_wheel_joint">
         <command_interface name="velocity" />
         <state_interface name="position" />

File: myagv_plus_description/urdf/myagv_plus.urdf.xacro (robot description, xacro)
@@ -4,4 +4,5 @@
   <xacro:arg name="namespace" default=""/>
   <xacro:arg name="use_sim" default="false" />
+  <xacro:property name="controller_config" value="$(arg controller_config)" />
   <xacro:property name="namespace" value="$(arg namespace)" />
   <xacro:property name="use_sim" value="$(arg use_sim)" />

Commit message: fix(myagv_plus_hardware_interfaces): add esp32 system

File: myagv_plus_description/urdf/common/ros2_control.urdf.xacro (robot description, xacro)
@@ -36,4 +36,31 @@
         <param name="can_id">0x04</param>
         <param name="mst_id">0x14</param>
+      </joint>
+    </ros2_control>
+  </xacro:macro>
+  <xacro:macro name="esp32_system" params="name:='esp32_system' namespace:=''">
+    <xacro:property name="ns" value="${namespace + '/' if namespace != '' else ''}" />
+    <ros2_control name="${ns}${name}" type="system">
+      <hardware>
+        <plugin>myagvplus_hardware_interfaces/Esp32Interface</plugin>
+        <param name="port">/dev/myagvplus_esp32</param>
+        <param name="baudrate">115200</param>
+      </hardware>
+      <sensor name="${ns}imu">
+        <state_interface name="orientation.x"/>
+        <state_interface name="orientation.y"/>
+        <state_interface name="orientation.z"/>
+        <state_interface name="orientation.w"/>
+        <state_interface name="angular_velocity.x"/>
+        <state_interface name="angular_velocity.y"/>
+        <state_interface name="angular_velocity.z"/>
+        <state_interface name="linear_acceleration.x"/>
+        <state_interface name="linear_acceleration.y"/>
+        <state_interface name="linear_acceleration.z"/>
+      </sensor>
+      <joint name="${ns}rgb_led">
+        <command_interface name="r"/>
+        <command_interface name="g"/>
+        <command_interface name="b"/>
       </joint>
     </ros2_control>
