Commit message: fix(myagv_plus_description): Update and fix xacro files

File: myagv_plus_description/urdf/robot/base.urdf.xacro (robot description, xacro)
@@ -2,25 +2,76 @@
 <robot xmlns:xacro="http://www.ros.org/wiki/xacro">
   <!-- base defining macro -->
-  <xacro:macro name="base" params="wheel_radius namespace">
-    <link name="${namespace}_base_link">
+  <xacro:macro name="base" params="wheel_radius">
+    <link name="base_footprint"/>
+    <joint name="base_joint" type="fixed">
+      <parent link="base_footprint"/>
+      <child link="base_link" />
+      <origin xyz="0 0 ${wheel_radius}" rpy="0 0 0"/>
+    </joint>
+    <link name="base_link">
       <visual>
         <geometry>
-          <cylinder radius="${wheel_radius}" length="0.1" />
+          <mesh filename="package://myagv_plus_description/meshes/base_link.stl"/>
         </geometry>
-        <origin xyz="0.0 0.0 0.05" rpy="0.0 0.0 0.0" />
+        <origin xyz="0.0 0.0 0.0" rpy="0.0 0.0 0.0" />
+        <material name="White">
+          <color rgba="1.0 1.0 1.0 1.0" />
+        </material>
+        <gazebo reference="base_link">
+          <material>Gazebo/White</material>
+        </gazebo>
       </visual>
       <collision>
         <geometry>
-          <cylinder radius="${wheel_radius}" length="0.1" />
+          <mesh filename="package://myagv_plus_description/meshes/base_link.stl"/>
         </geometry>
-        <origin xyz="0.0 0.0 0.05" rpy="0.0 0.0 0.0" />
+        <origin xyz="0.0 0.0 0.0" rpy="0.0 0.0 0.0" />
       </collision>
       <inertial>
-        <mass value="1.0" />
-        <inertia ixx="0.1" ixy="0.0" ixz="0.0"
-                  iyy="0.1" iyz="0.0"
-                  izz="0.1" />
+        <mass value="5" />
+        <inertia ixx="0.005" ixy="0.0"     ixz="0.0"
+                                iyy="0.005" iyz="0.0"
+                                              izz="0.005" />
+        <origin xyz="0.0 0.0 0.025" rpy="0.0 0.0 0.0" />
       </inertial>
     </link>
+    <link name="laser_link">
+      <visual>
+        <geometry>
+          <mesh filename="package://myagv_plus_description/meshes/laser_link.stl"/>
+        </geometry>
+        <origin xyz="0.0 0.0 0.0" rpy="0.0 0.0 0.0" />
+        <material name="White">
+          <color rgba="1.0 1.0 1.0 1.0" />
+        </material>
+        <gazebo reference="laser_link">
+          <material>Gazebo/White</material>
+        </gazebo>
+      </visual>
+      <collision>
+        <geometry>
+          <mesh filename="package://myagv_plus_description/meshes/laser_link.stl"/>
+        </geometry>
+        <origin xyz="0.0 0.0 0.0" rpy="0.0 0.0 0.0" />
+      </collision>
+      <inertial>
+        <mass value="0.2" />
+        <inertia ixx="0.0001" ixy="0.0"     ixz="0.0"
+                                iyy="0.0001" iyz="0.0"
+                                              izz="0.0001" />
+        <origin xyz="0.0 0.0 0.0" rpy="0.0 0.0 0.0" />
+      </inertial>
+    <link name="imu_link">
+    <joint name="imu_joint" type="fixed">
+      <origin xyz="-0.17181 -0.0270532 0.14928" rpy="0 0 1.5707" />
+      <parent link="base_link" />
+      <child link="imu_link" />
+    </joint>
+    <link name="camera_link">
+    <joint name="camera_joint" type="fixed">
+      <origin xyz="0.23191 0 0.14928" rpy="0 0 0" />
+      <parent link="base_link" />
+      <child link="camera_link" />
+    </joint>
   </xacro:macro>
 </robot>

File: myagv_plus_description/urdf/robot/wheel.urdf.xacro (robot description, xacro)
@@ -2,5 +2,5 @@
 <robot xmlns:xacro="http://www.ros.org/wiki/xacro">
   <!-- wheel defining macro -->
-  <xacro:macro name="wheel" params="side wheel_radius namespace">
+  <xacro:macro name="wheel" params="side wheel_radius">
     <xacro:property name="wheel_separation_x" value="0.106" />
     <xacro:property name="wheel_separation_y" value="0.192" />
@@ -10,9 +10,9 @@
     <xacro:property name="iyy" value="0.000067" />
     <xacro:property name="izz" value="0.000041" />
-    <xacro:property name="x" value="0.0" />
+    <!-- <xacro:property name="x" value="0.0" />
     <xacro:property name="y" value="0.0" />
     <xacro:property name="mesh" value="" />
     <xacro:property name="visual_rotation" value="0.0" />
-    <xacro:property name="fdir" value="1.0 0.0 0.0" />
+    <xacro:property name="fdir" value="1.0 0.0 0.0" /> -->
     <xacro:if value="${side == 'lf'}">
       <xacro:property name="x" value="${wheel_separation_x/2.0}" />
@@ -43,7 +43,7 @@
       <xacro:property name="fdir" value="1.0 -1.0 0.0" />
     </xacro:if>
-    <joint name="${namespace}${side}_wheel_joint" type="continuous">
-      <parent link="${namespace}base_link" />
-      <child link="${namespace}${side}_wheel_link" />
+    <joint name="${side}_wheel_joint" type="continuous">
+      <parent link="base_link" />
+      <child link="${side}_wheel_link" />
       <origin xyz="${x} ${y} 0.0" rpy="0.0 0.0 0.0" />
       <axis xyz="0.0 1.0 0.0" />
@@ -51,8 +51,8 @@
       <dynamics damping="0.001" friction="0.001" />
     </joint>
-    <link name="${namespace}${side}_wheel_link">
+    <link name="${side}_wheel_link">
       <visual>
         <geometry>
-          <mesh filename="${mesh}" scale="1.0 1.0 1.0" />
+          <mesh filename="${mesh}" />
         </geometry>
         <origin xyz="0.0 0.0 0.0" rpy="0.0 0.0 ${visual_rotation}" />
@@ -63,5 +63,5 @@
       <collision>
         <geometry>
-          <cylinder radius="${wheel_radius}" length="${wheel_thickness}" />
+          <mesh filename="${mesh}" />
         </geometry>
         <origin xyz="0.0 0.0 0.0" rpy="${pi/2} 0.0 0.0" />
@@ -74,5 +74,5 @@
       </inertial>
     </link>
-    <gazebo reference="${namespace}${side}_wheel_link" xmlns:ignition="http://ignitionrobotics.org/schema">
+    <gazebo reference="${side}_wheel_link" xmlns:ignition="http://ignitionrobotics.org/schema">
       <collision>
         <surface>

Commit message: fix(myagv_plus_description): fix URDF model and control code

File: myagv_plus_description/urdf/robot/base.urdf.xacro (robot description, xacro)
@@ -7,5 +7,5 @@
       <parent link="base_footprint"/>
       <child link="base_link" />
-      <origin xyz="0 0 ${wheel_radius}" rpy="0 0 0"/>
+      <origin xyz="0 0 0.0175" rpy="0 0 0"/>
     </joint>
     <link name="base_link">
@@ -63,12 +63,12 @@
       </inertial>
     </link>
-    <joint name="$lidar_joint" type="fixed">
-      <origin xyz="0.17891 0 0.20928" rpy="0 0 0" />
+    <joint name="lidar_joint" type="fixed">
+      <origin xyz="0.07471 0 0.07377" rpy="0 0 0" />
       <parent link="base_link" />
       <child link="laser_link" />
-  </joint>
+    </joint>
     <link name="imu_link" />
     <joint name="imu_joint" type="fixed">
-      <origin xyz="-0.17181 -0.0270532 0.14928" rpy="0 0 1.5707" />
+      <origin xyz="0.0 0.0 0.02" rpy="0 0 1.5707" />
       <parent link="base_link" />
       <child link="imu_link" />
@@ -76,5 +76,5 @@
     <link name="camera_link" />
     <joint name="camera_joint" type="fixed">
-      <origin xyz="0.23191 0 0.14928" rpy="0 0 0" />
+      <origin xyz="0.15991 0 0.051" rpy="0 0 0" />
       <parent link="base_link" />
       <child link="camera_link" />

File: myagv_plus_description/urdf/robot/wheel.urdf.xacro (robot description, xacro)
@@ -3,6 +3,6 @@
   <!-- wheel defining macro -->
   <xacro:macro name="wheel" params="side wheel_radius">
-    <xacro:property name="wheel_separation_x" value="0.34362" />
-    <xacro:property name="wheel_separation_y" value="0.3598" />
+    <xacro:property name="wheel_separation_x" value="0.233" />
+    <xacro:property name="wheel_separation_y" value="0.23884" />
     <xacro:property name="wheel_thickness" value="0.036" />
     <xacro:property name="mass" value="0.074" />
@@ -14,5 +14,5 @@
       <xacro:property name="y" value="${wheel_separation_y/2.0}" />
       <xacro:property name="mesh" value="package://myagv_plus_description/meshes/wheel_fl_link.stl" />
-      <xacro:property name="visual_rotation" value="${pi}" />
+      <xacro:property name="visual_rotation" value="${0.0}" />
       <xacro:property name="fdir" value="1.0 -1.0 0.0" />
     </xacro:if>
@@ -21,5 +21,5 @@
       <xacro:property name="y" value="${-wheel_separation_y/2.0}" />
       <xacro:property name="mesh" value="package://myagv_plus_description/meshes/wheel_fr_link.stl" />
-      <xacro:property name="visual_rotation" value="${pi}" />
+      <xacro:property name="visual_rotation" value="${0.0}" />
       <xacro:property name="fdir" value="1.0 1.0 0.0" />
     </xacro:if>
@@ -41,7 +41,7 @@
       <parent link="base_link" />
       <child link="${side}_wheel_link" />
-      <origin xyz="${x} ${y} 0.0" rpy="0.0 0.0 0.0" />
+      <origin xyz="${x} ${y} 0.019524" rpy="0.0 0.0 0.0" />
       <axis xyz="0.0 1.0 0.0" />
-      <limit effort="1.5" velocity="24.0" />
+      <limit effort="1.35" velocity="40.0" />
       <dynamics damping="0.001" friction="0.001" />
     </joint>

Commit message: fix(myagv_plus_controller): Modify controller speed and wheel spacing

File: myagv_plus_description/urdf/robot/base.urdf.xacro (robot description, xacro)
@@ -64,5 +64,5 @@
     </link>
     <joint name="lidar_joint" type="fixed">
-      <origin xyz="0.07471 0 0.07377" rpy="0 0 0" />
+      <origin xyz="0.07471 0 0.07377" rpy="0 0 3.14159" />
       <parent link="base_link" />
       <child link="laser_link" />
