Commit message: fix(hardware_interfaces): Update the hardware components of the ROS2 controller.

File: myagv_plus_description/urdf/robot/wheel.urdf.xacro (robot description, xacro)
@@ -3,6 +3,6 @@
   <!-- wheel defining macro -->
   <xacro:macro name="wheel" params="side wheel_radius">
-    <xacro:property name="wheel_separation_x" value="0.106" />
-    <xacro:property name="wheel_separation_y" value="0.192" />
+    <xacro:property name="wheel_separation_x" value="0.34362" />
+    <xacro:property name="wheel_separation_y" value="0.3598" />
     <xacro:property name="wheel_thickness" value="0.036" />
     <xacro:property name="mass" value="0.074" />

Commit message: fix(myagv_plus_description): Fix the collision property in urdf

File: myagv_plus_description/urdf/robot/wheel.urdf.xacro (robot description, xacro)
@@ -60,5 +60,5 @@
           <mesh filename="${mesh}" />
         </geometry>
-        <origin xyz="0.0 0.0 0.0" rpy="${pi/2} 0.0 0.0" />
+        <origin xyz="0.0 0.0 0.0" rpy="0.0 0.0 0.0" />
       </collision>
       <inertial>
